File: hardware/BioAmp-EXG-Pill.sch (KiCad schematic (older format))
At the start: 27 parts, among them J1 BioAmp Output, J2 BioAmp Input, U1 TL074, U2 LOGO_UDLABS

Commit message: redesigned PCB for manufacture MedTech style
Parts:
- U2: symbol udlabs:LOGO_UDLABS -> BioAmp-EXG-Pill-rescue:LOGO_UDLABS-udlabs
Changed lines of the file:
@@
 contact@upsidedownlabs.tech
 $Comp
-L udlabs:LOGO_UDLABS U2
+L BioAmp-EXG-Pill-rescue:LOGO_UDLABS-udlabs U2
 U 1 1 612DF07B
 P 6950 940
