File: hardware/BioAmp-EXG-Pill_1206.sch (KiCad schematic (older format))
At the start: 29 parts, among them J1 BioAmp Output, J2 BioAmp Input, J3 AudioJack3_SwitchTR, J4 AudioJack3_SwitchTR, U1 TL074, U2 LOGO_UDLABS

Commit message: complete redesign for FeatherWint
Parts:
- added BOARD1: FeaterWing Board, BioAmp:WeatherWing_empty, symbol BioAmp-EXG-Pill-rescue:LOGOS
- added D1, D2, D3, D4, D5, D6: LED, BioAmp:LED_0805_2012Metric_Pad1.15x1.40mm_HandSolder, symbol Device:LED_Small
- added F1: feather long, BioAmp:PinHeader_1x16_FeatherLong, symbol Connector_Generic:Conn_01x16
- added F2: feather short, BioAmp:PinHeader_1x12_FeatherShort, symbol Connector_Generic:Conn_01x12
- added JP3, JP4: Jumper_NO_Small, BioAmp:PinHeader_1x02_P2.54mm_Vertical, symbol Device:Jumper_NO_Small
- added JP5: SolderJumper_2_Bridged, BioAmp:SolderJumper-2_P1.3mm_Bridged, symbol Jumper:SolderJumper_2_Bridged
- added JP6: SolderJumper_2_Open, BioAmp:SolderJumper-2_P1.3mm_Open_RoundedPad1.0x1.5mm, symbol Jumper:SolderJumper_2_Open
- added LOGO2: LOGO_Coconut, BioAmp:Coconut_logo, symbol BioAmp-EXG-Pill-rescue:LOGOS
- added LOGO3: CoconutResearch, BioAmp:LOGO-CoconutText, symbol BioAmp-EXG-Pill-rescue:LOGOS
- added R16: R, BioAmp:R_1206_dusjagr, symbol Device:R
- added R17: 1K, BioAmp:R_1206_dusjagr, symbol Device:R
- added R18: 2K2, BioAmp:R_1206_dusjagr, symbol Device:R
- C6: footprint BioAmp:C_1210_dusjagr -> BioAmp:C_1206_dusjagr
- J2: value BioAmp Input -> StressRelief Output; footprint BioAmp:BioAmpInput_PinHeader_1x03_P2.54mm_Vertical -> BioAmp:PinHeader_1x03_StressRelief
- J3: value AudioJack3_SwitchTR -> AudioJack_Mono; footprint BioAmp:AUDIO-Jack_3.5mm_5Pin -> BioAmp:PJ301M-12_dusjagr_3d; symbol Connector:AudioJack3_SwitchTR -> Connector:AudioJack2_SwitchT
- J4: value AudioJack3_SwitchTR -> AudioJack_TRS
- JP1: footprint Jumper:SolderJumper-3_P1.3mm_Open_RoundedPad1.0x1.5mm -> BioAmp:SolderJumper-3_P1.3mm_Open_RoundedPad1.0x1.5mm
- JP2: footprint Jumper:SolderJumper-2_P1.3mm_Open_RoundedPad1.0x1.5mm -> BioAmp:SolderJumper-2_P1.3mm_Open_RoundedPad1.0x1.5mm
- LOGO1: renamed from U2; footprint udlabs:EXG -> BioAmp:LOGO-UpsideDownLabs-EXG
- U1: footprint 1Channel_PiezoAmp:SO-14_5.3x10.2mm_P1.27mm -> BioAmp:SO-14_5.3x10.2mm_P1.27mm
Connections:
- net DRL: no longer J2.1 (Pin_1)
- net GND: now also J2.2 (Pin_2), F1.13 (Pin_13), R16.1, R18.2
- net IN+: no longer J2.2 (Pin_2)
- net IN-: no longer J2.3 (Pin_3)
- net OUT: now also J2.1 (Pin_1), JP3.2, R17.2
- net VCC: now also J2.3 (Pin_3), JP5.1 (A), JP6.1 (A)
- net at R1.2, R4.2, R8.1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: now also JP4.1
- net at R1.1, R5.2, R9.1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: now also JP4.2
- net at C2.1, JP2.1 (A): now also JP3.1
- new net: D1.1 (K), D2.1 (K), D3.1 (K), D4.1 (K), D5.1 (K), D6.1 (K), R16.2
- new net +3V3: F1.15 (Pin_15)
- new net A0: F1.12 (Pin_12), R17.1, R18.1
- new net A1: F1.11 (Pin_11)
- new net A2: F1.10 (Pin_10)
- new net A3: F1.9 (Pin_9)
- new net A4: F1.8 (Pin_8)
- new net A5: F1.7 (Pin_7)
- new net AREF: F1.14 (Pin_14)
- new net EN: F2.11 (Pin_11)
- new net F0: F2.3 (Pin_3)
- new net F1: D1.2 (A), F2.4 (Pin_4)
- new net F2: D2.2 (A), F2.5 (Pin_5)
- new net F3: D3.2 (A), F2.6 (Pin_6)
- new net F4: D4.2 (A), F2.7 (Pin_7)
- new net F5: D5.2 (A), F2.8 (Pin_8)
- new net F6: D6.2 (A), F2.9 (Pin_9)
- new net LDO2: F1.1 (Pin_1), JP6.2 (B)
- new net MISO: F1.4 (Pin_4)
- new net MOSI: F1.5 (Pin_5)
- new net RX: F1.3 (Pin_3)
- new net SCK: F1.6 (Pin_6)
- new net SCL: F2.2 (Pin_2)
- new net SDA: F2.1 (Pin_1)
- new net TX: F1.2 (Pin_2)
- new net VBAT: F2.12 (Pin_12)
- new net VUSB: F2.10 (Pin_10), JP5.2 (B)
- new net ~RST: F1.16 (Pin_16)
Other:
- note added: "FeatherBoard / LEDs"
- note added: "Jack Input"
- note added: "UPlabs: contact@upsidedownlabs.tech"
- note added: "dusjagr: marc@dusseiller.ch"
- note removed: "contact@upsidedownlabs.tech"
- moved on the sheet: C1, C2, C3, C4, C5, C6, C8, J1, J4, JP1, LOGO1, R1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
